File: kbxIrBlaster.kicad_pcb (KiCad board)
At the start: 2 copper layers, 79.4 x 33 mm, 51 parts, among them J1 Conn_02x04_Odd_Even, J2 Conn_01x06, J3 Conn_01x15, J4 Conn_01x15, J5 Barrel_Jack_Switch, J6 USB_B_Micro, Q1 2N7002, Q2 2N7002, Q3 2N7002, Q4 2N7002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

Commit message: PCB refinements
Parts:
- added JP7: SolderJumper_2_Open, Jumper:SolderJumper-2_P1.3mm_Open_RoundedPad1.0x1.5mm, B.Cu at (151.8, 78.1)
- JP1, JP2, JP6: footprint Jumper:SolderJumper-2_P1.3mm_Open_Pad1.0x1.5mm -> Jumper:SolderJumper-2_P1.3mm_Open_RoundedPad1.0x1.5mm
- JP3, JP4, JP5: footprint Jumper:SolderJumper-3_P1.3mm_Open_Pad1.0x1.5mm -> Jumper:SolderJumper-3_P1.3mm_Open_RoundedPad1.0x1.5mm
- JP8: renamed from JP7; footprint Jumper:SolderJumper-3_P1.3mm_Open_Pad1.0x1.5mm -> Jumper:SolderJumper-3_P1.3mm_Open_RoundedPad1.0x1.5mm
- moved REF** 11.2 mm to (182.9, 66.7)
Connections:
- JP5 pad 1: GPIO15 -> GPIO16
- JP6 pad 2: GPIO2 -> GPIO15
Routing:
- net GPIO16: track 11.4 -> 38.8 mm
- net GPIO15: track 38.9 -> 22.8 mm
- net +BATT: track 15.7 -> 18.2 mm
- net GPIO2: track 33.3 -> 35.0 mm
- net +5V: track 80.7 -> 82.2 mm, vias 0 -> 1
Other:
- board text added: "433 MHz Transmitter"
- board text removed: "+"
- board text removed: "-"
- board text removed: "6 VDC max input 1 A max"
- board text removed: "IO2"
- board text removed: "LED 2"
- board text removed: "Outputs"
- board text removed: "Post-diode V+"
- board text removed: "U1"
- board text removed: "U2"
