File: kbxIrBlaster.sch (KiCad schematic (older format))
At the start: 50 parts, among them J1 Conn_02x04_Odd_Even, J2 Conn_01x06, J3 Conn_01x15, J4 Conn_01x15, J5 Barrel_Jack_Switch, J6 USB_B_Micro, Q1 2N7002, Q2 2N7002, Q3 2N7002, Q4 2N7002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

Commit message: PCB refinements
Parts:
- added JP7: SolderJumper_2_Open, Jumper:SolderJumper-2_P1.3mm_Open_RoundedPad1.0x1.5mm, symbol Jumper:SolderJumper_2_Open
- JP1, JP2, JP6: footprint Jumper:SolderJumper-2_P1.3mm_Open_Pad1.0x1.5mm -> Jumper:SolderJumper-2_P1.3mm_Open_RoundedPad1.0x1.5mm
- JP3, JP4, JP5: footprint Jumper:SolderJumper-3_P1.3mm_Open_Pad1.0x1.5mm -> Jumper:SolderJumper-3_P1.3mm_Open_RoundedPad1.0x1.5mm
- JP8: renamed from JP7; footprint Jumper:SolderJumper-3_P1.3mm_Open_Pad1.0x1.5mm -> Jumper:SolderJumper-3_P1.3mm_Open_RoundedPad1.0x1.5mm
Connections:
- net +5V: now also JP7.2 (B)
- net +BATT: now also JP7.1 (A)
- net GPIO15: now also JP6.2 (B); no longer JP5.1 (A)
- net GPIO16: now also JP5.1 (A)
- net GPIO2: no longer JP6.2 (B)
Changed lines of the file:
@@
 	1750 5350 1550 5350
 Wire Wire Line
-	1550 4950 1550 5350
-Wire Wire Line
-	2350 4950 2350 5350
+	1550 4950 1550 5000
+Wire Wire Line
+	2350 4950 2350 5000
 Connection ~ 2350 5750
 Wire Wire Line
@@
 	2950 5350 3350 5350
 $Comp
-L Jumper:SolderJumper_3_Open JP7
+L Jumper:SolderJumper_3_Open JP8
 U 1 1 5E394047
 P 4600 5100
-F 0 "JP7" H 4600 5305 50  0000 C CNN
+F 0 "JP8" H 4600 5305 50  0000 C CNN
 F 1 "SolderJumper_3_Open" H 4600 5214 50  0000 C CNN
-F 2 "Jumper:SolderJumper-3_P1.3mm_Open_Pad1.0x1.5mm" H 4600 5100 50  0001 C CNN
+F 2 "Jumper:SolderJumper-3_P1.3mm_Open_RoundedPad1.0x1.5mm" H 4600 5100 50  0001 C CNN
 F 3 "~" H 4600 5100 50  0001 C CNN
 	1    4600 5100
@@
 F 0 "JP1" V 4604 2318 50  0000 L CNN
 F 1 "SolderJumper_2_Open" V 4695 2318 50  0000 L CNN
-F 2 "Jumper:SolderJumper-2_P1.3mm_Open_Pad1.0x1.5mm" H 4650 2250 50  0001 C CNN
+F 2 "Jumper:SolderJumper-2_P1.3mm_Open_RoundedPad1.0x1.5mm" H 4650 2250 50  0001 C CNN
 F 3 "~" H 4650 2250 50  0001 C CNN
 	1    4650 2250
@@
 F 0 "JP2" V 5604 2318 50  0000 L CNN
 F 1 "SolderJumper_2_Open" V 5695 2318 50  0000 L CNN
-F 2 "Jumper:SolderJumper-2_P1.3mm_Open_Pad1.0x1.5mm" H 5650 2250 50  0001 C CNN
+F 2 "Jumper:SolderJumper-2_P1.3mm_Open_RoundedPad1.0x1.5mm" H 5650 2250 50  0001 C CNN
 F 3 "~" H 5650 2250 50  0001 C CNN
 	1    5650 2250
@@
 F 0 "JP3" H 8050 2455 50  0000 C CNN
 F 1 "SolderJumper_3_Open" H 8050 2364 50  0000 C CNN
-F 2 "Jumper:SolderJumper-3_P1.3mm_Open_Pad1.0x1.5mm" H 8050 2250 50  0001 C CNN
+F 2 "Jumper:SolderJumper-3_P1.3mm_Open_RoundedPad1.0x1.5mm" H 8050 2250 50  0001 C CNN
 F 3 "~" H 8050 2250 50  0001 C CNN
 	1    8050 2250
@@
 F 0 "JP4" H 9000 2455 50  0000 C CNN
 F 1 "SolderJumper_3_Open" H 9000 2364 50  0000 C CNN
-F 2 "Jumper:SolderJumper-3_P1.3mm_Open_Pad1.0x1.5mm" H 9000 2250 50  0001 C CNN
+F 2 "Jumper:SolderJumper-3_P1.3mm_Open_RoundedPad1.0x1.5mm" H 9000 2250 50  0001 C CNN
 F 3 "~" H 9000 2250 50  0001 C CNN
 	1    9000 2250
@@
 F 0 "JP5" H 9950 2455 50  0000 C CNN
 F 1 "SolderJumper_3_Open" H 9950 2364 50  0000 C CNN
-F 2 "Jumper:SolderJumper-3_P1.3mm_Open_Pad1.0x1.5mm" H 9950 2250 50  0001 C CNN
+F 2 "Jumper:SolderJumper-3_P1.3mm_Open_RoundedPad1.0x1.5mm" H 9950 2250 50  0001 C CNN
 F 3 "~" H 9950 2250 50  0001 C CNN
 	1    9950 2250
@@
 	3550 4750 3550 5700
 Connection ~ 3550 5700
-Text GLabel 9950 1850 1    50   BiDi ~ 0
+Text GLabel 9100 4300 2    50   BiDi ~ 0
 GPIO15
-Text GLabel 9000 1850 1    50   BiDi ~ 0
-GPIO2
 $Comp
 L Interface_Optical:TSOP382xx U1
@@
 F 0 "JP6" V 8854 4368 50  0000 L CNN
 F 1 "SolderJumper_2_Open" V 8945 4368 50  0000 L CNN
-F 2 "Jumper:SolderJumper-2_P1.3mm_Open_Pad1.0x1.5mm" H 8900 4300 50  0001 C CNN
+F 2 "Jumper:SolderJumper-2_P1.3mm_Open_RoundedPad1.0x1.5mm" H 8900 4300 50  0001 C CNN
 F 3 "~" H 8900 4300 50  0001 C CNN
 	1    8900 4300
@@
 	-1   0    0    -1
 $EndComp
-Text GLabel 9100 4300 2    50   BiDi ~ 0
+Text GLabel 9000 1850 1    50   BiDi ~ 0
 GPIO2
 Wire Wire Line
@@
 Text Notes 7200 3300 0    50   Italic 0
 Note: Calculate appropriate values for R1 through R4 based on LED forward current!\n LEDs are in series, so use (Vf * 2) — e.g.: R = (Vin - 0.5 - (Vf * 2)) / If\n Vin may be up to 6 volts but subtract 0.5 volts because of D9/D10/D12.\n 2N7002 FETs can handle up to 200 mA each; FETs capable of more current may be used if required.
+Text GLabel 9950 1850 1    50   BiDi ~ 0
+GPIO16
+$Comp
+L Jumper:SolderJumper_2_Open JP7
+U 1 1 5F7DE179
+P 1900 5000
+F 0 "JP7" V 1854 5068 50  0000 L CNN
+F 1 "SolderJumper_2_Open" V 1945 5068 50  0000 L CNN
+F 2 "Jumper:SolderJumper-2_P1.3mm_Open_RoundedPad1.0x1.5mm" H 1900 5000 50  0001 C CNN
+F 3 "~" H 1900 5000 50  0001 C CNN
+	1    1900 5000
+	1    0    0    -1
+$EndComp
+Wire Wire Line
+	1750 5000 1550 5000
+Connection ~ 1550 5000
+Wire Wire Line
+	1550 5000 1550 5350
+Wire Wire Line
+	2050 5000 2350 5000
+Connection ~ 2350 5000
+Wire Wire Line
+	2350 5000 2350 5350
 $EndSCHEMATC
